File: GTB.sch (KiCad schematic (older format))
At the start: 7 parts, among them U1 7555

Commit message: Added README.md
Parts:
- BT1: symbol Battery -> Battery-RESCUE-GTB
- D1: symbol LED -> LED-RESCUE-GTB
Changed lines of the file:
@@
 EESchema Schematic File Version 2
+LIBS:GTB-rescue
 LIBS:power
 LIBS:device
@@
 Connection ~ 5600 2550
 $Comp
-L LED D1
+L LED-RESCUE-GTB D1
 U 1 1 5772F917
 P 6150 4050
@@
 	4800 3950 4800 4100
 $Comp
-L Battery BT1
+L Battery-RESCUE-GTB BT1
 U 1 1 5772FC7A
 P 4050 3350
